File: Pathfinder.kicad_pcb (KiCad board)
At the start: 2 copper layers, 10 parts, among them SW1 SW_Push, SW2 SW_Push, SW3 SW_Push, U1 XIAO-RP2040-DIP

Commit message: finished PCB
Parts:
- R1, R2, R3: footprint Resistor_THT:R_Axial_DIN0207_L6.3mm_D2.5mm_P7.62mm_Horizontal -> Resistor_THT:R_Axial_DIN0204_L3.6mm_D1.6mm_P5.08mm_Horizontal
- SW1, SW2, SW3: footprint Button_Switch_THT:SW_PUSH_6mm -> Button_Switch_Keyboard:SW_Cherry_MX_1.00u_PCB
- moved SW1 42.4 mm to (131.8, 152.1)
- moved SW3 23.0 mm to (131.8, 110.6)
- moved SW2 11.2 mm to (131.8, 131.5)
Routing:
- net button3: track 46.1 -> 17.8 mm
- net button1: track 35.6 -> 55.2 mm
- net GND: track 150.8 -> 144.0 mm
- net button2: track 43.0 -> 36.7 mm
- net LED2: track 18.6 -> 21.1 mm
- net LED3: track 12.7 -> 15.2 mm
- net LED1: track 25.0 -> 26.1 mm
Other:
- board outline added: 56 x 117.3 mm
